File: rasp_tv_spi_version.kicad_sch (KiCad schematic)
At the start: 11 parts, among them J1 Raspberry_Pi_2_3, J6 PAM8302-input, J7 PAM8302-output, J8 SPEAKER, J9 5V_USB, SW1 SW_Push_DPDT, U1 TFT_320x240

Commit message: make pcb routing
Parts:
- removed J6: PAM8302-input, Connector_PinHeader_2.54mm:PinHeader_1x05_P2.54mm_Vertical, symbol Connector:Conn_01x05_Pin
- removed J7: PAM8302-output, Connector_PinHeader_2.54mm:PinHeader_1x02_P2.54mm_Vertical, symbol Connector:Conn_01x02_Pin
- removed J9: 5V_USB, Connector_Wire:SolderWirePad_1x01_SMD_1.5x3mm, symbol Connector:Conn_01x02_Pin
- added J2: Conn_01x09, Connector_PinHeader_2.54mm:PinHeader_1x09_P2.54mm_Vertical, symbol Connector_Generic:Conn_01x09
- added J3: Conn_01x09, Connector_PinHeader_2.54mm:PinHeader_1x09_P2.54mm_Vertical_SMD_Pin1Left, symbol Connector_Generic:Conn_01x09
- added J4: AUODIO_IN, Connector_PinHeader_2.54mm:PinHeader_1x05_P2.54mm_Vertical_SMD_Pin1Left, symbol Connector_Generic:Conn_01x05
- added J5: SPEAKER, Connector_PinHeader_2.54mm:PinHeader_1x02_P2.54mm_Horizontal, symbol Connector_Generic:Conn_01x02
- added J6, J7: AUDIO_OUT, Connector_PinSocket_2.54mm:PinSocket_1x02_P2.54mm_Vertical_SMD_Pin1Left, symbol Connector_Generic:Conn_01x02
- added U2: PAM8302AAD, Module:PAM, symbol Amplifier_Audio:PAM8302AAD_module
- J1: footprint Connector_PinHeader_2.54mm:PinHeader_2x20_P2.54mm_Vertical -> Connector_PinSocket_2.54mm:PinSocket_2x20_P2.54mm_Vertical
- J8: value SPEAKER -> Conn_01x02_Pin; footprint Connector_Hirose:Hirose_DF13C_CL535-0402-2-51_1x02-1MP_P1.25mm_Vertical -> Connector_PinHeader_2.54mm:PinHeader_1x02_P2.54mm_Horizontal
- SW1: footprint Button_Switch_THT:SW_Push_2P2T_Toggle_CK_PVA2OAH5xxxxxxV2 -> Button_Switch_THT:SW_DPDT_XLX
Connections:
- net +3.3V: now also J2.9 (Pin_9), J3.8 (Pin_8); no longer U1.8 (LED)
- net +5V: now also J4.4 (Pin_4)
- net CS_8_GPIO: now also J2.7 (Pin_7), J3.7 (Pin_7)
- net DC_24_GPIO: now also J2.5 (Pin_5), J3.5 (Pin_5)
- net GND: now also J2.8 (Pin_8), J3.9 (Pin_9), J4.2 (Pin_2), J4.5 (Pin_5), U2.4 (IN-)
- net MISO_0_09_GPIO: now also J2.1 (Pin_1), J3.1 (Pin_1)
- net MOSI_0_10_GPIO: now also J2.4 (Pin_4), J3.4 (Pin_4)
- net RESET_25_GPIO: now also J2.6 (Pin_6), J3.6 (Pin_6)
- net SCK_0_11_GPIO: now also J2.3 (Pin_3), J3.3 (Pin_3)
- net AUDIO_IN: now reaches RV1.2
- net AUDIO_IN: now also J4.1 (Pin_1), U2.5 (IN+)
- net at SW1.3 (C): now also J8.1 (Pin_1)
- net at SW1.4 (A): now also J8.2 (Pin_2)
- net BACKLIGHT_23_GPIO: now reaches J1.16 (GPIO23)
- net BACKLIGHT_23_GPIO: now also U1.8 (LED), J2.2 (Pin_2), J3.2 (Pin_2)
- new net: J5.2 (Pin_2), J7.1 (Pin_1), U2.6 (OUT+)
- new net: J5.1 (Pin_1), J6.2 (Pin_2), U2.7 (OUT-)
- no-connect marks 0 -> 1
Other:
- moved on the sheet: C1, R1, R2, RV1, SW1, U1

Commit message: finish board with 2.8 spi
Parts:
- added J9: Raspberry_Pi_2_3, Connector_PinSocket_2.54mm:PinSocket_2x20_P2.54mm_Vertical, symbol Connector:Raspberry_Pi_2_3
- J6, J7: footprint Connector_PinSocket_2.54mm:PinSocket_1x02_P2.54mm_Vertical_SMD_Pin1Left -> Connector_PinHeader_2.54mm:PinHeader_1x02_P2.54mm_Vertical_SMD_Pin1Left
Connections:
- net +3.3V: now also J9.1 (3V3), J9.17 (3V3)
- net +5V: now also J9.2 (5V), J9.4 (5V)
- net BACKLIGHT_23_GPIO: now also J9.16 (GPIO23)
- net CS_8_GPIO: now also J9.24 (~{CE0}/GPIO8)
- net DC_24_GPIO: now also J9.18 (GPIO24)
- net GND: now also J9.14 (GND), J9.20 (GND), J9.25 (GND), J9.30 (GND), J9.34 (GND), J9.39 (GND), J9.6 (GND), J9.9 (GND)
- net MISO_0_09_GPIO: now also J9.21 (MISO0/GPIO9)
- net MOSI_0_10_GPIO: now also J9.19 (MOSI0/GPIO10)
- net PWM_19_GPIO: now also J9.35 (GPIO19/MISO1)
- net RESET_25_GPIO: now also J9.22 (GPIO25)
- net SCK_0_11_GPIO: now also J9.23 (SCLK0/GPIO11)
- no-connect marks 1 -> 3

Commit message: ready for factory
Parts:
- removed J4: AUODIO_IN, Connector_PinHeader_2.54mm:PinHeader_1x05_P2.54mm_Vertical_SMD_Pin1Left, symbol Connector_Generic:Conn_01x05
- removed J6, J7: AUDIO_OUT, Connector_PinHeader_2.54mm:PinHeader_1x02_P2.54mm_Vertical_SMD_Pin1Left, symbol Connector_Generic:Conn_01x02
- added J4: Conn_01x05_Pin, Connector_PinHeader_2.54mm:PinHeader_1x05_P2.54mm_Vertical, symbol Connector:Conn_01x05_Pin
- added J6: OUT1, Connector_PinHeader_2.54mm:PinHeader_1x01_P2.54mm_Vertical, symbol Connector:Conn_01x01_Pin
- added J7: OUT2, Connector_PinHeader_2.54mm:PinHeader_1x01_P2.54mm_Vertical, symbol Connector:Conn_01x01_Pin
- J5: footprint Connector_PinHeader_2.54mm:PinHeader_1x02_P2.54mm_Horizontal -> Connector_Hirose:Hirose_DF3EA-02P-2V_1x02-1MP_P2.00mm_Vertical
- J8: footprint Connector_PinHeader_2.54mm:PinHeader_1x02_P2.54mm_Horizontal -> Connector_Wire:SolderWire-0.1sqmm_1x02_P3.6mm_D0.4mm_OD1mm
Connections:
- net +5V: now also J4.4 (Pin_4)
- net AUDIO_IN: now also J4.1 (Pin_1)
- net GND: now also J4.2 (Pin_2), J4.5 (Pin_5)
- net at J5.2 (Pin_2), U2.6 (OUT+): now also J7.1 (Pin_1)
- net at J5.1 (Pin_1), U2.7 (OUT-): now also J6.1 (Pin_1)
- no-connect marks 3 -> 0
Changed lines of the file:
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@@
 		(color 0 0 0 0)
 	)
-	(no_connect
-		(at 247.65 45.72)
-	)
-	(no_connect
-		(at 247.65 54.61)
-	)
-	(no_connect
-		(at 259.08 33.02)
-	)
 	(wire
 		(pts
@@
 	)
 	(symbol
-		(lib_id "Connector_Generic:Conn_01x05")
-		(at 264.16 33.02 0)
+		(lib_id "Connector:Conn_01x01_Pin")
+		(at 242.57 52.07 0)
 		(unit 1)
 		(exclude_from_sim no)
@@
 		(on_board yes)
 		(dnp no)
-		(fields_autoplaced yes)
-		(property "Reference" "J4"
-			(at 266.7 31.7499 0)
+		(property "Reference" "J7"
+			(at 240.284 52.07 0)
 			(effects
 				(font
 					(size 1.27 1.27)
 				)
-				(justify left)
 			)
 		)
-		(property "Value" "AUODIO_IN"
-			(at 266.7 34.2899 0)
+		(property "Value" "OUT2"
+			(at 242.316 54.102 0)
 			(effects
 				(font
 					(size 1.27 1.27)
 				)
-				(justify left)
 			)
 		)
-		(property "Footprint" "Connector_PinHeader_2.54mm:PinHeader_1x05_P2.54mm_Vertical_SMD_Pin1Left"
-			(at 264.16 33.02 0)
+		(property "Footprint" "Connector_PinHeader_2.54mm:PinHeader_1x01_P2.54mm_Vertical"
+			(at 242.57 52.07 0)
 			(effects
 				(font
@@
 		)
 		(property "Datasheet" "~"
-			(at 264.16 33.02 0)
+			(at 242.57 52.07 0)
 			(effects
 				(font
@@
 			)
 		)
-		(property "Description" "Generic connector, single row, 01x05, script generated (kicad-library-utils/schlib/autogen/connector/)"
-			(at 264.16 33.02 0)
+		(property "Description" "Generic connector, single row, 01x01, script generated"
+			(at 242.57 52.07 0)
 			(effects
 				(font
@@
 			)
 		)
-		(pin "3"
-		)
-		(pin "2"
-		)
-		(pin "5"
-		)
 		(pin "1"
 		)
-		(pin "4"
-		)
 		(instances
 			(project ""
 				(path "/076c14dd-ffa4-4616-978a-d572d1838aa1"
-					(reference "J4")
+					(reference "J7")
 					(unit 1)
 				)
@@
 	)
 	(symbol
+		(lib_id "Connector:Conn_01x05_Pin")
+		(at 264.16 33.02 0)
+		(mirror y)
+		(unit 1)
+		(exclude_from_sim no)
+		(in_bom yes)
+		(on_board yes)
+		(dnp no)
+		(property "Reference" "J4"
+			(at 263.525 22.86 0)
+			(effects
+				(font
+					(size 1.27 1.27)
+				)
+			)
+		)
+		(property "Value" "Conn_01x05_Pin"
+			(at 263.525 25.4 0)
+			(effects
+				(font
+					(size 1.27 1.27)
+				)
+			)
+		)
+		(property "Footprint" "Connector_PinHeader_2.54mm:PinHeader_1x05_P2.54mm_Vertical"
+			(at 264.16 33.02 0)
+			(effects
+				(font
+					(size 1.27 1.27)
+				)
+				(hide yes)
+			)
+		)
+		(property "Datasheet" "~"
+			(at 264.16 33.02 0)
+			(effects
+				(font
+					(size 1.27 1.27)
+				)
+				(hide yes)
+			)
+		)
+		(property "Description" "Generic connector, single row, 01x05, script generated"
+			(at 264.16 33.02 0)
+			(effects
+				(font
+					(size 1.27 1.27)
+				)
+				(hide yes)
+			)
+		)
+		(pin "2"
+		)
+		(pin "3"
+		)
+		(pin "4"
+		)
+		(pin "5"
+		)
+		(pin "1"
+		)
+		(instances
+			(project ""
+				(path "/076c14dd-ffa4-4616-978a-d572d1838aa1"
+					(reference "J4")
+					(unit 1)
+				)
+			)
+		)
+	)
+	(symbol
 		(lib_id "power:+5V")
 		(at 63.5 29.21 0)
@@
 		)
 		(property "Footprint" "Button_Switch_THT:SW_DPDT_XLX"
-			(at 226.06 114.3 0)
+			(at 230.886 101.092 0)
 			(effects
 				(font
@@
 	)
 	(symbol
-		(lib_id "Connector_Generic:Conn_01x02")
-		(at 242.57 52.07 0)
-		(mirror y)
-		(unit 1)
-		(exclude_from_sim no)
-		(in_bom yes)
-		(on_board yes)
-		(dnp no)
-		(property "Reference" "J7"
-			(at 239.268 55.118 0)
-			(effects
-				(font
-					(size 1.27 1.27)
-				)
-			)
-		)
-		(property "Value" "AUDIO_OUT"
-			(at 243.078 57.658 0)
-			(effects
-				(font
-					(size 1.27 1.27)
-				)
-			)
-		)
-		(property "Footprint" "Connector_PinHeader_2.54mm:PinHeader_1x02_P2.54mm_Vertical_SMD_Pin1Left"
-			(at 282.956 83.82 0)
-			(effects
-				(font
-					(size 1.27 1.27)
-				)
-			)
-		)
-		(property "Datasheet" "~"
-			(at 242.57 52.07 0)
-			(effects
-				(font
-					(size 1.27 1.27)
-				)
-				(hide yes)
-			)
-		)
-		(property "Description" "Generic connector, single row, 01x02, script generated (kicad-library-utils/schlib/autogen/connector/)"
-			(at 242.57 52.07 0)
-			(effects
-				(font
-					(size 1.27 1.27)
-				)
-				(hide yes)
-			)
-		)
-		(pin "1"
-		)
-		(pin "2"
-		)
-		(instances
-			(project "rasp_tv_spi_version"
-				(path "/076c14dd-ffa4-4616-978a-d572d1838aa1"
-					(reference "J7")
-					(unit 1)
-				)
-			)
-		)
-	)
-	(symbol
 		(lib_id "Connector:Conn_01x02_Pin")
 		(at 243.84 116.84 0)
@@
 			)
 		)
-		(property "Footprint" "Connector_PinHeader_2.54mm:PinHeader_1x02_P2.54mm_Horizontal"
+		(property "Footprint" "Connector_Wire:SolderWire-0.1sqmm_1x02_P3.6mm_D0.4mm_OD1mm"
 			(at 245.618 138.938 0)
 			(effects
@@
 	)
 	(symbol
-		(lib_id "Connector_Generic:Conn_01x02")
-		(at 242.57 45.72 0)
-		(mirror y)
+		(lib_id "Connector:Conn_01x01_Pin")
+		(at 242.57 48.26 0)
 		(unit 1)
 		(exclude_from_sim no)
@@
 		(dnp no)
 		(property "Reference" "J6"
-			(at 242.316 42.418 0)
+			(at 240.792 44.196 0)
 			(effects
 				(font
@@
 			)
 		)
-		(property "Value" "AUDIO_OUT"
-			(at 235.458 42.926 0)
+		(property "Value" "OUT1"
+			(at 239.776 47.498 0)
 			(effects
 				(font
@@
 			)
 		)
-		(property "Footprint" "Connector_PinHeader_2.54mm:PinHeader_1x02_P2.54mm_Vertical_SMD_Pin1Left"
-			(at 299.72 18.288 0)
+		(property "Footprint" "Connector_PinHeader_2.54mm:PinHeader_1x01_P2.54mm_Vertical"
+			(at 242.57 48.26 0)
 			(effects
 				(font
@@
 		)
 		(property "Datasheet" "~"
-			(at 242.57 45.72 0)
+			(at 242.57 48.26 0)
 			(effects
 				(font
@@
 			)
 		)
-		(property "Description" "Generic connector, single row, 01x02, script generated (kicad-library-utils/schlib/autogen/connector/)"
-			(at 242.57 45.72 0)
+		(property "Description" "Generic connector, single row, 01x01, script generated"
+			(at 242.57 48.26 0)
 			(effects
 				(font
@@
 		(pin "1"
 		)
-		(pin "2"
-		)
 		(instances
-			(project "rasp_tv_spi_version"
+			(project ""
 				(path "/076c14dd-ffa4-4616-978a-d572d1838aa1"
 					(reference "J6")
@@
 			)
 		)
-		(property "Footprint" "Connector_PinHeader_2.54mm:PinHeader_1x02_P2.54mm_Horizontal"
+		(property "Footprint" "Connector_Hirose:Hirose_DF3EA-02P-2V_1x02-1MP_P2.00mm_Vertical"
 			(at 265.43 52.07 0)
 			(effects
